Commit message: missing /

File: description/robot_core.xacro (robot description, xacro)
@@ -6,11 +6,11 @@
     <material name ="orange">
         <color rgba ="1 0.3 0.1 1"/>
-    <material>
+    </material>
     <material name="blue">
         <color rgba ="0.2 0.2 1 1"/>
-    <material>
+    </material>
     <material name ="black">
         <color rgba ="0 0 0 1"/>
-    <material>
+    </material>
      <link name ="base_link">
      </link>
@@ -25,5 +25,5 @@
             <geometry>
                 <box size="0.3 0.3 0.15"/>
-            <geometry>
+            </geometry>
             <material name="white"/>
         </visual>

Commit message: cylinder shape is changed

File: description/robot_core.xacro (robot description, xacro)
@@ -24,5 +24,5 @@
             <origin xyz="0.15 0 0.075"/>
             <geometry>
-                <box size="0.3 0.3 0.15"/>
+                <cylinder size="0.3 0 1"/>
             </geometry>
             <material name="white"/>

Commit message: updated chassis with wheels

File: description/robot_core.xacro (robot description, xacro)
@@ -24,8 +24,38 @@
             <origin xyz="0.15 0 0.075"/>
             <geometry>
-                <cylinder size="0.3 0 1"/>
+                <box size="0.3 0.3 0.15"/>
             </geometry>
             <material name="white"/>
         </visual>
     </link>
+    <!--LEFT WHEEL LINK-->
+    <joint name="left_wheel_joint" type="continous">
+        <parent link="base_link"/>
+        <child link="left_wheel"/>
+        <origin xyz="0 0.175 0" rpy="-${pi/2} 0 0"
+        <axis xyz ="0 0 1"/>
+    </joint>
+    <link name ="left_wheel">
+        <visual>
+            <geometry>
+                <cylinder radius="0.05" length="0.04"/>
+            </geometry>
+        <material name ="blue"/>
+        </visual>
+    </link>
+    <!--RIGHT WHEEL LINK-->
+    <joint name="right_wheel_joint" type="continous">
+        <parent link="base_link"/>
+        <child link="right_wheel"/>
+        <origin xyz="0 -0.175 0" rpy="${pi/2} 0 0"
+        <axis xyz ="0 0 1"/>
+    </joint>
+    <link name ="right_wheel">
+        <visual>
+            <geometry>
+                <cylinder radius="0.05" length="0.04"/>
+            </geometry>
+        <material name ="blue"/>
+        </visual>
+    </link>
 </robot>

Commit message: updated chasssi

File: description/robot_core.xacro (robot description, xacro)
@@ -30,8 +30,8 @@
     </link>
     <!--LEFT WHEEL LINK-->
-    <joint name="left_wheel_joint" type="continous">
+    <joint name="left_wheel_joint" type="continuous">
         <parent link="base_link"/>
         <child link="left_wheel"/>
-        <origin xyz="0 0.175 0" rpy="-${pi/2} 0 0"
+        <origin xyz="0 0.175 0" rpy="-${pi/2} 0 0"/>
         <axis xyz ="0 0 1"/>
     </joint>
@@ -45,8 +45,8 @@
     </link>
     <!--RIGHT WHEEL LINK-->
-    <joint name="right_wheel_joint" type="continous">
+    <joint name="right_wheel_joint" type="continuous">
         <parent link="base_link"/>
         <child link="right_wheel"/>
-        <origin xyz="0 -0.175 0" rpy="${pi/2} 0 0"
+        <origin xyz="0 -0.175 0" rpy="${pi/2} 0 0"/>
         <axis xyz ="0 0 1"/>
     </joint>

Commit message: u

File: description/robot_core.xacro (robot description, xacro)
@@ -59,3 +59,19 @@
         </visual>
     </link>
+    <!--CASTOR VALL ROLLER LINK-->
+        <!--RIGHT WHEEL LINK-->
+    <joint name="castor_wheel_joint" type="fixed">
+        <parent link="chassis"/>
+        <child link="castor_wheel"/>
+        <origin xyz="0.24 0 0"u rpy="0 0 0"/>
+        <axis xyz ="0 0 1"/>
+    </joint>
+    <link name ="castor_wheel">
+        <visual>
+            <geometry>
+                <sphere radius="0.05"/>
+            </geometry>
+        <material name ="black"/>
+        </visual>
+    </link>
 </robot>

Commit message: u

File: description/robot_core.xacro (robot description, xacro)
@@ -64,5 +64,5 @@
         <parent link="chassis"/>
         <child link="castor_wheel"/>
-        <origin xyz="0.24 0 0"u rpy="0 0 0"/>
+        <origin xyz="0.24 0 0" rpy="0 0 0"/>
         <axis xyz ="0 0 1"/>
     </joint>

Commit message: collision enabled

File: description/robot_core.xacro (robot description, xacro)
@@ -28,4 +28,10 @@
             <material name="white"/>
         </visual>
+        <collision>
+            <origin xyz="0.15 0 0.075"/>
+            <geometry>
+                <box size="0.3 0.3 0.15"/>
+            </geometry>
+        </collision>
     </link>
     <!--LEFT WHEEL LINK-->
@@ -43,4 +49,9 @@
         <material name ="blue"/>
         </visual>
+        <collision>
+            <geometry>
+                <cylinder radius="0.05" length="0.04"/>
+            </geometry>
+        </collision>
     </link>
     <!--RIGHT WHEEL LINK-->
@@ -58,4 +69,9 @@
         <material name ="blue"/>
         </visual>
+        <collision>
+            <geometry>
+                <cylinder radius="0.05" length="0.04"/>
+            </geometry>
+        </collision>
     </link>
     <!--CASTOR VALL ROLLER LINK-->
@@ -74,4 +90,9 @@
         <material name ="black"/>
         </visual>
+        <collision>
+            <geometry>
+                <sphere radius="0.05"/>
+            </geometry>
+        </collision>
     </link>
 </robot>

Commit message: gg

File: description/robot_core.xacro (robot description, xacro)
@@ -35,46 +35,5 @@
         </collision>
     </link>
-    <!--LEFT WHEEL LINK-->
-    <joint name="left_wheel_joint" type="continuous">
-        <parent link="base_link"/>
-        <child link="left_wheel"/>
-        <origin xyz="0 0.175 0" rpy="-${pi/2} 0 0"/>
-        <axis xyz ="0 0 1"/>
-    </joint>
-    <link name ="left_wheel">
-        <visual>
-            <geometry>
-                <cylinder radius="0.05" length="0.04"/>
-            </geometry>
-        <material name ="blue"/>
-        </visual>
-        <collision>
-            <geometry>
-                <cylinder radius="0.05" length="0.04"/>
-            </geometry>
-        </collision>
-    </link>
-    <!--RIGHT WHEEL LINK-->
-    <joint name="right_wheel_joint" type="continuous">
-        <parent link="base_link"/>
-        <child link="right_wheel"/>
-        <origin xyz="0 -0.175 0" rpy="${pi/2} 0 0"/>
-        <axis xyz ="0 0 1"/>
-    </joint>
-    <link name ="right_wheel">
-        <visual>
-            <geometry>
-                <cylinder radius="0.05" length="0.04"/>
-            </geometry>
-        <material name ="blue"/>
-        </visual>
-        <collision>
-            <geometry>
-                <cylinder radius="0.05" length="0.04"/>
-            </geometry>
-        </collision>
-    </link>
     <!--CASTOR VALL ROLLER LINK-->
-        <!--RIGHT WHEEL LINK-->
     <joint name="castor_wheel_joint" type="fixed">
         <parent link="chassis"/>

Commit message: gg

File: description/robot_core.xacro (robot description, xacro)
@@ -35,4 +35,24 @@
         </collision>
     </link>
+    <!--LEFT WHEEL LINK-->
+    <joint name="left_wheel_joint" type="continuous">
+        <parent link="base_link"/>
+        <child link="left_wheel"/>
+        <origin xyz="0 0.175 0" rpy="-${pi/2} 0 0"/>
+        <axis xyz ="0 0 1"/>
+    </joint>
+    <link name ="left_wheel">
+        <visual>
+            <geometry>
+                <cylinder radius="0.05" length="0.04"/>
+            </geometry>
+        <material name ="blue"/>
+        </visual>
+        <collision>
+            <geometry>
+                <cylinder radius="0.05" length="0.04"/>
+            </geometry>
+        </collision>
+    </link>gg
     <!--CASTOR VALL ROLLER LINK-->
     <joint name="castor_wheel_joint" type="fixed">

Commit message: gg

File: description/robot_core.xacro (robot description, xacro)
@@ -54,5 +54,5 @@
             </geometry>
         </collision>
-    </link>gg
+    </link>
     <!--CASTOR VALL ROLLER LINK-->
     <joint name="castor_wheel_joint" type="fixed">

Commit message: y

File: description/robot_core.xacro (robot description, xacro)
@@ -35,12 +35,12 @@
         </collision>
     </link>
-    <!--LEFT WHEEL LINK-->
-    <joint name="left_wheel_joint" type="continuous">
+    <!--RIGHT WHEEL LINK-->
+    <joint name="right_wheel_joint" type="continuous">
         <parent link="base_link"/>
-        <child link="left_wheel"/>
-        <origin xyz="0 0.175 0" rpy="-${pi/2} 0 0"/>
+        <child link="right_wheel"/>
+        <origin xyz="0 -0.175 0" rpy="${pi/2} 0 0"/>
         <axis xyz ="0 0 1"/>
     </joint>
-    <link name ="left_wheel">
+    <link name ="right_wheel">
         <visual>
             <geometry>

Commit message: first

File: description/robot_core.xacro (robot description, xacro)
@@ -35,4 +35,24 @@
         </collision>
     </link>
+    <!--LEFT WHEEL LINK-->
+    <joint name="left_wheel_joint" type="continuous">
+        <parent link="base_link"/>
+        <child link="left_wheel"/>
+        <origin xyz="0 0.175 0" rpy="-${pi/2} 0 0"/>
+        <axis xyz ="0 0 1"/>
+    </joint>
+    <link name ="left_wheel">
+        <visual>
+            <geometry>
+                <cylinder radius="0.05" length="0.04"/>
+            </geometry>
+        <material name ="blue"/>
+        </visual>
+        <collision>
+            <geometry>
+                <cylinder radius="0.05" length="0.04"/>
+            </geometry>
+        </collision>
+    </link>
     <!--RIGHT WHEEL LINK-->
     <joint name="right_wheel_joint" type="continuous">
@@ -62,16 +82,2 @@
         <axis xyz ="0 0 1"/>
     </joint>
-    <link name ="castor_wheel">
-        <visual>
-            <geometry>
-                <sphere radius="0.05"/>
-            </geometry>
-        <material name ="black"/>
-        </visual>
-        <collision>
-            <geometry>
-                <sphere radius="0.05"/>
-            </geometry>
-        </collision>
-    </link>
-</robot>

Commit message: castor fixed

File: description/robot_core.xacro (robot description, xacro)
@@ -82,3 +82,11 @@
         <axis xyz ="0 0 1"/>
     </joint>
+    <link name ="castor_wheel">
+        <visual>
+            <geometry>
+                <sphere radius="0.05"/>
+            </geometry>
+        <material name ="black"/>
+        </visual>
+    </link>
 </robot>

Commit message: gg

File: description/robot_core.xacro (robot description, xacro)
@@ -75,18 +75,3 @@
         </collision>
     </link>
-    <!--CASTOR VALL ROLLER LINK-->
-    <joint name="castor_wheel_joint" type="fixed">
-        <parent link="chassis"/>
-        <child link="castor_wheel"/>
-        <origin xyz="0.24 0 0" rpy="0 0 0"/>
-        <axis xyz ="0 0 1"/>
-    </joint>
-    <link name ="castor_wheel">
-        <visual>
-            <geometry>
-                <sphere radius="0.05"/>
-            </geometry>
-        <material name ="black"/>
-        </visual>
-    </link>
 </robot>

Commit message: gg

File: description/robot_core.xacro (robot description, xacro)
@@ -35,24 +35,4 @@
         </collision>
     </link>
-    <!--LEFT WHEEL LINK-->
-    <joint name="left_wheel_joint" type="continuous">
-        <parent link="base_link"/>
-        <child link="left_wheel"/>
-        <origin xyz="0 0.175 0" rpy="-${pi/2} 0 0"/>
-        <axis xyz ="0 0 1"/>
-    </joint>
-    <link name ="left_wheel">
-        <visual>
-            <geometry>
-                <cylinder radius="0.05" length="0.04"/>
-            </geometry>
-        <material name ="blue"/>
-        </visual>
-        <collision>
-            <geometry>
-                <cylinder radius="0.05" length="0.04"/>
-            </geometry>
-        </collision>
-    </link>
     <!--RIGHT WHEEL LINK-->
     <joint name="right_wheel_joint" type="continuous">
@@ -75,3 +55,18 @@
         </collision>
     </link>
+    <!--CASTOR VALL ROLLER LINK-->
+    <joint name="castor_wheel_joint" type="fixed">
+        <parent link="chassis"/>
+        <child link="castor_wheel"/>
+        <origin xyz="0.24 0 0" rpy="0 0 0"/>
+        <axis xyz ="0 0 1"/>
+    </joint>
+    <link name ="castor_wheel">
+        <visual>
+            <geometry>
+                <sphere radius="0.05"/>
+            </geometry>
+        <material name ="black"/>
+        </visual>
+    </link>
 </robot>

Commit message: no rpy

File: description/robot_core.xacro (robot description, xacro)
@@ -39,5 +39,5 @@
         <parent link="base_link"/>
         <child link="right_wheel"/>
-        <origin xyz="0 -0.175 0" rpy="${pi/2} 0 0"/>
+        <origin xyz="0 -0.175 0" />
         <axis xyz ="0 0 1"/>
     </joint>
@@ -47,5 +47,5 @@
                 <cylinder radius="0.05" length="0.04"/>
             </geometry>
-        <material name ="blue"/>
+            <material name ="blue"/>
         </visual>
         <collision>

Commit message: fixed

File: description/robot_core.xacro (robot description, xacro)
@@ -36,5 +36,5 @@
     </link>
     <!--RIGHT WHEEL LINK-->
-    <joint name="right_wheel_joint" type="continuous">
+    <joint name="right_wheel_joint" type="fixed">
         <parent link="base_link"/>
         <child link="right_wheel"/>

Commit message: conintous left wheel

File: description/robot_core.xacro (robot description, xacro)
@@ -36,8 +36,8 @@
     </link>
     <!--RIGHT WHEEL LINK-->
-    <joint name="right_wheel_joint" type="fixed">
+    <joint name="right_wheel_joint" type="continuous">
         <parent link="base_link"/>
         <child link="right_wheel"/>
-        <origin xyz="0 -0.175 0" />
+        <origin xyz="0 -0.175 0" rpy = "0 0 0"/>
         <axis xyz ="0 0 1"/>
     </joint>

Commit message: h

File: description/robot_core.xacro (robot description, xacro)
@@ -36,23 +36,23 @@
     </link>
     <!--RIGHT WHEEL LINK-->
-    <joint name="right_wheel_joint" type="continuous">
-        <parent link="base_link"/>
-        <child link="right_wheel"/>
-        <origin xyz="0 -0.175 0" rpy = "0 0 0"/>
-        <axis xyz ="0 0 1"/>
-    </joint>
-    <link name ="right_wheel">
-        <visual>
-            <geometry>
-                <cylinder radius="0.05" length="0.04"/>
-            </geometry>
-            <material name ="blue"/>
-        </visual>
-        <collision>
-            <geometry>
-                <cylinder radius="0.05" length="0.04"/>
-            </geometry>
-        </collision>
-    </link>
+<joint name="right_wheel_joint" type="continuous">
+    <parent link="base_link"/>
+    <child link="right_wheel"/>
+    <origin xyz="0 -0.175 0" rpy="0 0 0"/>
+    <axis xyz="0 0 1"/>
+</joint>
+<link name="right_wheel">
+    <visual>
+        <geometry>
+            <cylinder radius="0.05" length="0.04"/>
+        </geometry>
+        <material name="blue"/>
+    </visual>
+    <collision>
+        <geometry>
+            <cylinder radius="0.05" length="0.04"/>
+        </geometry>
+    </collision>
+</link>
     <!--CASTOR VALL ROLLER LINK-->
     <joint name="castor_wheel_joint" type="fixed">

Commit message: no collision

File: description/robot_core.xacro (robot description, xacro)
@@ -28,10 +28,4 @@
             <material name="white"/>
         </visual>
-        <collision>
-            <origin xyz="0.15 0 0.075"/>
-            <geometry>
-                <box size="0.3 0.3 0.15"/>
-            </geometry>
-        </collision>
     </link>
     <!--RIGHT WHEEL LINK-->
@@ -39,5 +33,5 @@
     <parent link="base_link"/>
     <child link="right_wheel"/>
-    <origin xyz="0 -0.175 0" rpy="0 0 0"/>
+    <origin xyz="0 0.175 0" rpy="-{pi/2} 0 0"/>
     <axis xyz="0 0 1"/>
 </joint>
@@ -49,9 +43,4 @@
         <material name="blue"/>
     </visual>
-    <collision>
-        <geometry>
-            <cylinder radius="0.05" length="0.04"/>
-        </geometry>
-    </collision>
 </link>
     <!--CASTOR VALL ROLLER LINK-->

Commit message: number

File: description/robot_core.xacro (robot description, xacro)
@@ -33,5 +33,5 @@
     <parent link="base_link"/>
     <child link="right_wheel"/>
-    <origin xyz="0 0.175 0" rpy="-{pi/2} 0 0"/>
+    <origin xyz="0 0.175 0" rpy="-{1.5708} 0 0"/>
     <axis xyz="0 0 1"/>
 </joint>

Commit message: n

File: description/robot_core.xacro (robot description, xacro)
@@ -33,5 +33,5 @@
     <parent link="base_link"/>
     <child link="right_wheel"/>
-    <origin xyz="0 0.175 0" rpy="-{1.5708} 0 0"/>
+    <origin xyz="0 0.175 0" rpy="0 0 0"/>
     <axis xyz="0 0 1"/>
 </joint>
@@ -48,5 +48,5 @@
         <parent link="chassis"/>
         <child link="castor_wheel"/>
-        <origin xyz="0.24 0 0" rpy="0 0 0"/>
+        <origin xyz="0.24 0 0" rpy="-1.5708 0 0"/>
         <axis xyz ="0 0 1"/>
     </joint>

Commit message: left and right

File: description/robot_core.xacro (robot description, xacro)
@@ -33,8 +33,22 @@
     <parent link="base_link"/>
     <child link="right_wheel"/>
-    <origin xyz="0 0.175 0" rpy="0 0 0"/>
+    <origin xyz="0 0.175 0" rpy="-${pi/2} 0 0"/>
     <axis xyz="0 0 1"/>
 </joint>
 <link name="right_wheel">
+    <visual>
+        <geometry>
+            <cylinder radius="0.05" length="0.04"/>
+        </geometry>
+        <material name="blue"/>
+    </visual>
+</link>
+<joint name="left_wheel_joint" type="continuous">
+    <parent link="base_link"/>
+    <child link="left_wheel"/>
+    <origin xyz="0 -0.175 0" rpy="${pi/2} 0 0"/>
+    <axis xyz="0 0 -1"/>
+</joint>
+<link name="left_wheel">
     <visual>
         <geometry>

Commit message: g

File: description/robot_core.xacro (robot description, xacro)
@@ -33,5 +33,5 @@
     <parent link="base_link"/>
     <child link="right_wheel"/>
-    <origin xyz="0 0.175 0" rpy="-${pi/2} 0 0"/>
+    <origin xyz="0 0.175 0" rpy="-1.5078 0 0"/>
     <axis xyz="0 0 1"/>
 </joint>
@@ -47,5 +47,5 @@
     <parent link="base_link"/>
     <child link="left_wheel"/>
-    <origin xyz="0 -0.175 0" rpy="${pi/2} 0 0"/>
+    <origin xyz="0 -0.175 0" rpy="1.5708 0 0"/>
     <axis xyz="0 0 -1"/>
 </joint>

Commit message: ff

File: description/robot_core.xacro (robot description, xacro)
@@ -30,5 +30,5 @@
     </link>
     <!--RIGHT WHEEL LINK-->
-<joint name="right_wheel_joint" type="continuous">
+<joint name="right_wheel_joint" type="fixed">
     <parent link="base_link"/>
     <child link="right_wheel"/>
@@ -44,5 +44,5 @@
     </visual>
 </link>
-<joint name="left_wheel_joint" type="continuous">
+<joint name="left_wheel_joint" type="fixed">
     <parent link="base_link"/>
     <child link="left_wheel"/>

Commit message: continuous

File: description/robot_core.xacro (robot description, xacro)
@@ -30,5 +30,5 @@
     </link>
     <!--RIGHT WHEEL LINK-->
-<joint name="right_wheel_joint" type="fixed">
+<joint name="right_wheel_joint" type="continuous">
     <parent link="base_link"/>
     <child link="right_wheel"/>
@@ -44,5 +44,5 @@
     </visual>
 </link>
-<joint name="left_wheel_joint" type="fixed">
+<joint name="left_wheel_joint" type="continuous">
     <parent link="base_link"/>
     <child link="left_wheel"/>

Commit message: c

File: description/robot_core.xacro (robot description, xacro)
@@ -62,5 +62,5 @@
         <parent link="chassis"/>
         <child link="castor_wheel"/>
-        <origin xyz="0.24 0 0" rpy="-1.5708 0 0"/>
+        <origin xyz="0.24 0 0" rpy="0 0 0"/>
         <axis xyz ="0 0 1"/>
     </joint>

Commit message: collision enabled

File: description/robot_core.xacro (robot description, xacro)
@@ -28,4 +28,10 @@
             <material name="white"/>
         </visual>
+        <collision>
+            <origin xyz="0.15 0 0.075"/>
+            <geometry>
+                <box size="0.3 0.3 0.15"/>
+            </geometry>
+        </collision>
     </link>
     <!--RIGHT WHEEL LINK-->
@@ -43,4 +49,9 @@
         <material name="blue"/>
     </visual>
+    <collision>
+        <geometry>
+            <cylinder radius="0.05" length="0.04"/>
+        </geometry>
+    </collision>
 </link>
 <joint name="left_wheel_joint" type="continuous">
@@ -57,4 +68,9 @@
         <material name="blue"/>
     </visual>
+    <collision>
+        <geometry>
+            <cylinder radius="0.05" length="0.04"/>
+        </geometry>
+    </collision>
 </link>
     <!--CASTOR VALL ROLLER LINK-->
@@ -72,4 +88,10 @@
         <material name ="black"/>
         </visual>
+        <collision>
+            <geometry>
+                <sphere radius="0.05"/>
+            </geometry>
+        <material name ="black"/>
+        </collision>
     </link>
 </robot>

Commit message: colliison more

File: description/robot_core.xacro (robot description, xacro)
@@ -92,5 +92,4 @@
                 <sphere radius="0.05"/>
             </geometry>
-        <material name ="black"/>
         </collision>
     </link>
